File: dcc-sniffer-arduino-shield.kicad_pcb (KiCad board)
At the start: 2 copper layers, 18.3 x 52.8 mm, 10 parts, among them J1 MV132, U1 6N137

Commit message: Mark DCC input pin D2.
Other:
- board text added: "D2 DCC input"
Changed lines of the file:
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@@
 		)
+	)
+	(gr_line
+		(start 155.702 94.234)
+		(end 156.464 93.472)
+		(stroke
+			(width 0.1)
+			(type default)
+		)
+		(layer "B.SilkS")
 	)
 	(gr_poly
@@
 		(layer "B.SilkS")
 	)
+	(gr_line
+		(start 155.448 93.98)
+		(end 155.448 94.488)
+		(stroke
+			(width 0.1)
+			(type default)
+		)
+		(layer "B.SilkS")
+	)
 	(gr_poly
 		(pts
@@
 		(layer "B.SilkS")
 	)
+	(gr_line
+		(start 155.448 94.488)
+		(end 155.956 94.488)
+		(stroke
+			(width 0.1)
+			(type default)
+		)
+		(layer "B.SilkS")
+	)
 	(gr_poly
 		(pts
@@
 		(layer "B.SilkS")
 	)
+	(gr_line
+		(start 156.464 93.472)
+		(end 155.448 94.488)
+		(stroke
+			(width 0.1)
+			(type default)
+		)
+		(layer "B.SilkS")
+	)
 	(gr_arc
 		(start 152.654 73.152)
@@
 		)
 	)
+	(gr_text "D2 DCC input"
+		(at 161.798 92.964 0)
+		(layer "B.SilkS")
+		(effects
+			(font
+				(size 1 1)
+				(thickness 0.1)
+			)
+			(justify mirror)
+		)
+	)
